Commit message: add gripper element and planned with gripper as chain

File: swiftpro/urdf/swift_model.xacro (robot description, xacro)
@@ -234,3 +234,20 @@
 	<origin xyz= "0.02741 0 0.02703" rpy = " 0 0 0" />
 </joint>
+<!-- gripper model -->
+<joint name="GripperToTcp" type="fixed">
+        <parent link="Link8"/>
+        <child link="Gripper"/>
+        <origin xyz="0.08 0.0 -0.10" rpy="3.1415 1.57 0"/>
+</joint>
+<link name="Gripper">
+        <visual>
+	    <origin xyz="0 0 0" rpy="0 0 0"/>
+            <geometry>
+      		<mesh filename="package://swiftpro/urdf/swift_links/unit_sphere.stl" scale="0.005 0.005 0.005"/>
+    	    </geometry>
+            <material name="">
+                <color rgba="0.3 0.3 0.3 1"/>
+            </material>
+        </visual>
+</link>
 </robot>
